File: hardware/cane-board/cane-board.kicad_pcb (KiCad board)
At the start: 4 copper layers, 46 x 100 mm, 95 parts, among them J1 12V battery, J10 Phone power, J11 Firmware, J2 Motor, J3 Kill switch, J4 Talk button, J5 Encoder, J6 I2C, J7 Buzzer motor, J8 Serial, Q1 AO3401A, Q2 AO3401A, Q3 AO3400A, Q4 AO3401A, SW1 Reset, SW2 Boot, SW3 Power, U1 ESP32-S3-WROOM-1-N4, U2 DRV8876PWPR, U3 K7805-1000R3, U4 AP2112K-3.3, U5 TPS2069CDBVR

Commit message: Cane board: fixes from an outside review
An outside review of 74ceffe found four things; each was checked
against the files and the makers' data before changing anything.

- Voltage dividers: 100k/22k put 4.4 V on IO2 and IO4 at the 24.4 V
  TVS clamp, over Espressif's 3.6 V limit, and pushed current into the
  processor with the power switch off. Now 1M/100k (R24 to R27, values
  only, all JLCPCB Basic): 2.2 V at the clamp, 1.15 V at a full pack,
  about 7 uA into an unpowered pin. Readings are battery / 11.
- Placement file: KiCad's origins (pin 1 for the connectors and the
  5 V module) and rotations went straight into it. make_fab.py now
  writes body centres and JLCPCB's rotations, read from JLCPCB's own
  footprint previews for each LCSC part: SOT-23 180, AP2112K and
  DRV8876 270, JST and XT30 180, the rest as KiCad. Generic tables
  would have turned U4 a quarter and C1 and J11 round.
- The pin-1 list for the placement preview had C1's stripe on the
  wrong side (it marks minus, on the right) and J11's A1 at the top
  left instead of the lower left.
- Watchdog: check_watchdog.py now also models the pin stopping high:
  asleep about 125 ms after, against about 60 ms stopped low. The
  firmware rules say to stop it low, define the rate as a 200 Hz
  square wave, and add arming and disarming order and the ADC range.

Copper, drill and silkscreen are unchanged. DRC 0 errors, 0
unconnected, board matches the schematic.
Parts:
- R24, R26: value 100k -> 1M
- R25, R27: value 22k -> 100k
Changed lines of the file:
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@@
 			)
 		)
-		(property "Value" "22k"
+		(property "Value" "100k"
 			(at 0 1.43 0)
 			(layer "F.Fab")
@@
 			)
 		)
-		(property "Value" "100k"
+		(property "Value" "1M"
 			(at 0 1.43 0)
 			(layer "F.Fab")
@@
 			)
 		)
-		(property "Value" "100k"
+		(property "Value" "1M"
 			(at 0 1.43 0)
 			(layer "F.Fab")
@@
 			)
 		)
-		(property "Value" "22k"
+		(property "Value" "100k"
 			(at 0 1.43 0)
 			(layer "F.Fab")
