File: hardware/cane-board/cane-board.kicad_sch (KiCad schematic)
At the start: 99 parts, among them J1 12V battery, J10 Phone power, J11 Firmware, J2 Motor, J3 Kill switch, J4 Talk button, J5 Encoder, J6 I2C, J7 Buzzer motor, J8 Serial, Q1 AO3401A, Q2 AO3401A, Q3 AO3400A, Q4 AO3401A, SW1 Reset, SW2 Boot, SW3 Power, U1 ESP32-S3-WROOM-1-N4, U2 DRV8876PWPR, U3 TPS54302DDCR, U4 AP2112K-3.3, U5 TPS2069CDBVR

Commit message: Cane board: 5 V module, XT30 motor socket, 2.2 A limit, hand-routed power
Replace the TPS54302 converter with a sealed K7805-1000R3 module and
move the power switch to the 3.3 V regulator's enable. Swap the motor
screw terminal for an upright XT30. Raise the current limit to 2.2 A
(R5 1.5k) to match the push the IBT-2 gave.

Draw the battery, motor-supply and motor tracks by hand (0.6-1.0 mm on
the outer layers) before autorouting, turn J2 and C4 round so those
tracks run straight, and tie stranded ground pads to a via. DRC: 0
errors, 0 unconnected. Update the BOM, cost, problems list and fab files.
Parts:
- removed C12: 100nF 50V, Capacitor_SMD:C_0603_1608Metric, symbol Device:C
- removed C25: 100pF, Capacitor_SMD:C_0603_1608Metric, symbol Device:C
- removed L1: 10uH 3.2A, Inductor_SMD:L_Changjiang_FNR6045S, symbol Device:L
- removed R13: 13k, Resistor_SMD:R_0603_1608Metric, symbol Device:R
- J2: footprint TerminalBlock_Phoenix:TerminalBlock_Phoenix_MKDS-1,5-2-5.08_1x02_P5.08mm_Horizontal -> Connector_AMASS:AMASS_XT30UPB-F_1x02_P5.0mm_Vertical; symbol Connector:Screw_Terminal_01x02 -> Connector_Generic:Conn_01x02; LCSC C474952 -> C108769; MPN KF128-5.08-2P-AA -> XT30UPB-F30.G.Y
- R5: value 2.2k -> 1.5k; LCSC C4190 -> C22843; MPN 0603WAF2201T5E -> 0603WAF1501T5E
- U3: value TPS54302DDCR -> K7805-1000R3; footprint Package_TO_SOT_SMD:SOT-23-6 -> Converter_DCDC:Converter_DCDC_RECOM_R-78E-0.5_THT; symbol Regulator_Switching:TPS54302 -> Converter_DCDC:R-78E5.0-1.0; LCSC C311983 -> C2992391; MPN TPS54302DDCR -> K7805-1000R3
Connections:
- net BUCK_SW is gone; now on net GND: U3.2 (GND)
- net +5V: now also U3.3 (OUT); no longer R12.1
- net +BATT: now also U3.1 (IN); no longer U3.3 (VIN)
- net GND: no longer U3.1 (GND)
- net VSYS: now also R12.1; no longer U4.3 (EN)
- removed net BUCK_BST: U3.6 (BOOT)
- net BUCK_EN renamed LDO_EN
- net LDO_EN: now also R12.2, U4.3 (EN); no longer U3.5 (EN)
- removed net BUCK_FB: R12.2, U3.4 (FB)
Other:
- note added: "12 V to 5 V: ready-made module"
- note added: "A sealed switching module (YLPTEC K7805-1000R3: 8-36 V in, 5 V 1 A out, pins 1 in, 2 ground, 3 out). The converter's layout is inside it, so the board's layout cannot spoil it."
- note added: "Current limit = 3.3 V / R5 / 1000 uA/A: 1.5k gives 2.2 A. All resistors 1%."
- note removed: "12 V to 5 V, 3 A"
- note removed: "Current limit = 3.3 V / R5 / 1000 uA/A: 2.2k gives 1.5 A. All resistors 1%."
- note removed: "SW3 to ground: converter off, so the processor is off. 100k and 13k give 5.2 V."
- moved on the sheet: R12, SW3

Commit message: Cane board: cooler kill-switch FET, keep braking, battery plug notes
R2 and R3 go from 47k and 100k to 10k and 13k, so Q2's gate gets 0.43
of the battery instead of a third: 3.9 V from a flat 9 V pack (about
0.3 W at the 2.2 A limit instead of 0.4 W) and 10.6 V at the TVS
clamp, still under its 12 V limit. The kill switch now carries about
0.5 mA and cuts the motor supply in about 2 ms. Values only: the routed
board, Gerbers and placement file are unchanged; DRC 0 errors, 0
unconnected, schematic and board values match.

PMODE stays on ground (PH/EN mode, so a commanded stop brakes). The
worm gear holds the wheel either way and a dropped link still sleeps
the driver, which coasts as the IBT-2 did; firmware can coast for FREE
by stopping the heartbeat. Recorded in the README and as decided in
POTENTIAL_PROBLEMS.md, with how to check the battery plug.

The schematic picture is redrawn from the current PDF; it still showed
the old TPS54302 converter.
Parts:
- R2: value 47k -> 10k; LCSC C25819 -> C25804; MPN 0603WAF4702T5E -> 0603WAF1002T5E
- R3: value 100k -> 13k; LCSC C25803 -> C22797; MPN 0603WAF1003T5E -> 0603WAF1302T5E
Other:
- note added: "Switch closed (or a jumper on J3): motor supply on, Q2's gate at 0.43 of the battery. Open, unplugged or a broken wire: off within about 2 ms. C26 keeps Q2 off at plug-in."
- note removed: "Switch closed (or a jumper on J3): motor supply on. Open, unplugged or a broken wire: off within about 6 ms. C26 keeps Q2 off while the battery is plugged in."
Changed lines of the file:
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@@
 		)
 	)
-	(text "Switch closed (or a jumper on J3): motor supply on. Open, unplugged or a\nbroken wire: off within about 6 ms. C26 keeps Q2 off while the battery is plugged in."
-		(exclude_from_sim no)
-		(at 129.54 101.6 0)
-		(effects
-			(font
-				(size 1.27 1.27)
-			)
-			(justify left bottom)
-		)
-	)
 	(text "Battery in: fuse and reverse-plug protection"
 		(exclude_from_sim no)
@@
 		)
 	)
+	(text "Switch closed (or a jumper on J3): motor supply on, Q2's gate at 0.43 of the battery.\nOpen, unplugged or a broken wire: off within about 2 ms. C26 keeps Q2 off at plug-in."
+		(exclude_from_sim no)
+		(at 129.54 101.6 0)
+		(effects
+			(font
+				(size 1.27 1.27)
+			)
+			(justify left bottom)
+		)
+	)
 	(text "Current limit = 3.3 V / R5 / 1000 uA/A: 1.5k gives 2.2 A. All resistors 1%."
 		(exclude_from_sim no)
@@
 			)
 		)
-		(property "Value" "47k"
+		(property "Value" "10k"
 			(at 171.958 46.99 0)
 			(show_name no)
@@
 			)
 		)
-		(property "MPN" "0603WAF4702T5E"
+		(property "MPN" "0603WAF1002T5E"
 			(at 170.18 45.72 0)
 			(hide yes)
@@
 			)
 		)
-		(property "LCSC" "C25819"
+		(property "LCSC" "C25804"
 			(at 170.18 45.72 0)
 			(hide yes)
@@
 			)
 		)
-		(property "Value" "100k"
+		(property "Value" "13k"
 			(at 212.598 46.99 0)
 			(show_name no)
@@
 			)
 		)
-		(property "MPN" "0603WAF1003T5E"
+		(property "MPN" "0603WAF1302T5E"
 			(at 210.82 45.72 0)
 			(hide yes)
@@
 			)
 		)
-		(property "LCSC" "C25803"
+		(property "LCSC" "C22797"
 			(at 210.82 45.72 0)
 			(hide yes)

Commit message: Cane board: fixes from an outside review
An outside review of 74ceffe found four things; each was checked
against the files and the makers' data before changing anything.

- Voltage dividers: 100k/22k put 4.4 V on IO2 and IO4 at the 24.4 V
  TVS clamp, over Espressif's 3.6 V limit, and pushed current into the
  processor with the power switch off. Now 1M/100k (R24 to R27, values
  only, all JLCPCB Basic): 2.2 V at the clamp, 1.15 V at a full pack,
  about 7 uA into an unpowered pin. Readings are battery / 11.
- Placement file: KiCad's origins (pin 1 for the connectors and the
  5 V module) and rotations went straight into it. make_fab.py now
  writes body centres and JLCPCB's rotations, read from JLCPCB's own
  footprint previews for each LCSC part: SOT-23 180, AP2112K and
  DRV8876 270, JST and XT30 180, the rest as KiCad. Generic tables
  would have turned U4 a quarter and C1 and J11 round.
- The pin-1 list for the placement preview had C1's stripe on the
  wrong side (it marks minus, on the right) and J11's A1 at the top
  left instead of the lower left.
- Watchdog: check_watchdog.py now also models the pin stopping high:
  asleep about 125 ms after, against about 60 ms stopped low. The
  firmware rules say to stop it low, define the rate as a 200 Hz
  square wave, and add arming and disarming order and the ADC range.

Copper, drill and silkscreen are unchanged. DRC 0 errors, 0
unconnected, board matches the schematic.
Parts:
- R24, R26: value 100k -> 1M; LCSC C25803 -> C22935; MPN 0603WAF1003T5E -> 0603WAF1004T5E
- R25, R27: value 22k -> 100k; LCSC C31850 -> C25803; MPN 0603WAF2202T5E -> 0603WAF1003T5E
Other:
- note added: "IO3, IO45, IO46 are boot-mode pins: left open. IO35 to IO37 are left open so a module with more memory also fits. Dividers 1M/100k: 2.2 V at the 24.4 V clamp, and only microamps into the processor when it is off."
- note removed: "IO3, IO45, IO46 are boot-mode pins: left open. IO35 to IO37 are left open so a module with more memory also fits."
Changed lines of the file:
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@@
 		)
 	)
-	(text "IO3, IO45, IO46 are boot-mode pins: left open.\nIO35 to IO37 are left open so a module with more memory also fits."
+	(text "IO3, IO45, IO46 are boot-mode pins: left open. IO35 to IO37 are left open so a module with more memory also fits.\nDividers 1M/100k: 2.2 V at the 24.4 V clamp, and only microamps into the processor when it is off."
 		(exclude_from_sim no)
 		(at 114.3 281.94 0)
@@
 			)
 		)
-		(property "Value" "22k"
+		(property "Value" "100k"
 			(at 133.858 265.43 0)
 			(show_name no)
@@
 			)
 		)
-		(property "MPN" "0603WAF2202T5E"
+		(property "MPN" "0603WAF1003T5E"
 			(at 132.08 264.16 0)
 			(hide yes)
@@
 			)
 		)
-		(property "LCSC" "C31850"
+		(property "LCSC" "C25803"
 			(at 132.08 264.16 0)
 			(hide yes)
@@
 			)
 		)
-		(property "Value" "100k"
+		(property "Value" "1M"
 			(at 121.158 265.43 0)
 			(show_name no)
@@
 			)
 		)
-		(property "MPN" "0603WAF1003T5E"
+		(property "MPN" "0603WAF1004T5E"
 			(at 119.38 264.16 0)
 			(hide yes)
@@
 			)
 		)
-		(property "LCSC" "C25803"
+		(property "LCSC" "C22935"
 			(at 119.38 264.16 0)
 			(hide yes)
@@
 			)
 		)
-		(property "Value" "100k"
+		(property "Value" "1M"
 			(at 166.878 265.43 0)
 			(show_name no)
@@
 			)
 		)
-		(property "MPN" "0603WAF1003T5E"
+		(property "MPN" "0603WAF1004T5E"
 			(at 165.1 264.16 0)
 			(hide yes)
@@
 			)
 		)
-		(property "LCSC" "C25803"
+		(property "LCSC" "C22935"
 			(at 165.1 264.16 0)
 			(hide yes)
@@
 			)
 		)
-		(property "Value" "22k"
+		(property "Value" "100k"
 			(at 179.578 265.43 0)
 			(show_name no)
@@
 			)
 		)
-		(property "MPN" "0603WAF2202T5E"
+		(property "MPN" "0603WAF1003T5E"
 			(at 177.8 264.16 0)
 			(hide yes)
@@
 			)
 		)
-		(property "LCSC" "C31850"
+		(property "LCSC" "C25803"
 			(at 177.8 264.16 0)
 			(hide yes)
